Commit message: Update open_manipulator_x description
Signed-off-by: Andrej Orsula <orsula.andrej@gmail.com>

File: open_manipulator_description/ros2_control/open_manipulator_x_position.ros2_control.xacro (robot description, xacro)
@@ -11,5 +11,5 @@
         <hardware>
           <xacro:if value="${use_fake_hardware}">
-            <plugin>fake_components/GenericSystem</plugin>
+            <plugin>mock_components/GenericSystem</plugin>
             <param name="fake_sensor_commands">${fake_sensor_commands}</param>
             <param name="state_following_offset">0.0</param>

File: open_manipulator_description/urdf/open_manipulator_x/open_manipulator_x.urdf.xacro (robot description, xacro)
@@ -40,4 +40,20 @@
     <origin xyz="0 0.025 -0.1263" rpy="-1.5708 -1.5708 0"/>
   </joint>
+  <joint name="$(arg prefix)end_effector_joint" type="fixed">
+    <parent link="$(arg prefix)link5"/>
+    <child link="$(arg prefix)end_effector_link"/>
+    <origin xyz="0.0817 0 0" rpy="0 0 0"/>
+  </joint>
+  <link name="$(arg prefix)end_effector_link">
+    <visual>
+      <origin xyz="0 0 0" rpy="0 0 0"/>
+      <geometry>
+        <box size="0.01 0.01 0.01"/>
+      </geometry>
+      <material name="red">
+        <color rgba="1.0 0.0 0.0 1"/>
+      </material>
+    </visual>
+  </link>
   <xacro:open_manipulator_x prefix="$(arg prefix)" />
   <xacro:open_manipulator_x_gazebo prefix="$(arg prefix)" />

File: open_manipulator_description/urdf/open_manipulator_x/open_manipulator_x_arm.urdf.xacro (robot description, xacro)
@@ -143,4 +143,10 @@
         </material>
       </visual>
+      <collision>
+        <origin xyz="0 0 0" rpy="0 0 0"/>
+        <geometry>
+          <mesh filename="${meshes_file_direction}/link5.stl" scale="0.001 0.001 0.001"/>
+        </geometry>
+      </collision>
        <inertial>
         <origin xyz="4.4206755e-02 3.6839985e-07 8.9142216e-03" />
